Commit message: Add joint accelerations and velocities. Add camera

File: ar_description/urdf/ar.ros2_control.xacro (robot description, xacro)
@@ -7,7 +7,13 @@
     calibrate
     joint_offset_parameters_file
+    joint_velocity_parameters_file
+    joint_acceleration_parameters_file
   ">
     <xacro:property name="joint_offset_parameters"
       value="${xacro.load_yaml(joint_offset_parameters_file)}"/>
+    <xacro:property name="joint_velocity_parameters"
+      value="${xacro.load_yaml(joint_velocity_parameters_file)}"/>
+    <xacro:property name="joint_acceleration_parameters"
+      value="${xacro.load_yaml(joint_acceleration_parameters_file)}"/>
     <ros2_control name="${name}" type="system">
       <hardware>
@@ -25,4 +31,6 @@
         </state_interface>
         <param name="position_offset">${joint_offset_parameters['joint_1']}</param>
+        <param name="joint_velocity">${joint_velocity_parameters['joint_1']}</param>
+        <param name="joint_acceleration">${joint_acceleration_parameters['joint_1']}</param>
       </joint>
       <joint name="joint_2">
@@ -35,4 +43,6 @@
         </state_interface>
         <param name="position_offset">${joint_offset_parameters['joint_2']}</param>
+        <param name="joint_velocity">${joint_velocity_parameters['joint_2']}</param>
+        <param name="joint_acceleration">${joint_acceleration_parameters['joint_2']}</param>
       </joint>
       <joint name="joint_3">
@@ -45,4 +55,6 @@
         </state_interface>
         <param name="position_offset">${joint_offset_parameters['joint_3']}</param>
+        <param name="joint_velocity">${joint_velocity_parameters['joint_3']}</param>
+        <param name="joint_acceleration">${joint_acceleration_parameters['joint_3']}</param>
       </joint>
       <joint name="joint_4">
@@ -55,4 +67,6 @@
         </state_interface>
         <param name="position_offset">${joint_offset_parameters['joint_4']}</param>
+        <param name="joint_velocity">${joint_velocity_parameters['joint_4']}</param>
+        <param name="joint_acceleration">${joint_acceleration_parameters['joint_4']}</param>
       </joint>
       <joint name="joint_5">
@@ -65,4 +79,6 @@
         </state_interface>
         <param name="position_offset">${joint_offset_parameters['joint_5']}</param>
+        <param name="joint_velocity">${joint_velocity_parameters['joint_5']}</param>
+        <param name="joint_acceleration">${joint_acceleration_parameters['joint_5']}</param>
       </joint>
       <joint name="joint_6">
@@ -75,4 +91,6 @@
         </state_interface>
         <param name="position_offset">${joint_offset_parameters['joint_6']}</param>
+        <param name="joint_velocity">${joint_velocity_parameters['joint_6']}</param>
+        <param name="joint_acceleration">${joint_acceleration_parameters['joint_6']}</param>
       </joint>
     </ros2_control>

File: ar_description/urdf/ar_camera_macro.xacro (robot description, xacro)
@@ -2,8 +2,21 @@
 <robot xmlns:xacro="http://wiki.ros.org/xacro">
   <xacro:macro name="ar_camera">
+    <joint name="camera_jump_joint" type="fixed">
+      <parent link="base_link" />
+      <child link="camera_jump_link" />
+      <origin xyz="0.01 -0.67 0.75" rpy="${0 * pi / 180} ${90 * pi / 180} ${0 * pi / 180}" />
+    </joint>
+    <link name="camera_jump_link">
+      <visual>
+        <geometry>
+          <box size="0.010 0.03 0.03" />
+        </geometry>
+        <color rgba="1 1 0 1"/>
+      </visual>
+    </link>
     <joint name="camera_joint" type="fixed">
-      <parent link="base_link" />
+      <parent link="camera_jump_link" />
       <child link="camera_link" />
-      <origin xyz="0 -0.35 1.0" rpy="0 ${pi/2} 0" />
+      <origin xyz="0 0 0" rpy="${0 * pi / 180} ${0 * pi / 180} ${27 * pi / 180}" />
     </joint>
     <link name="camera_link">
@@ -12,9 +25,9 @@
           <box size="0.010 0.03 0.03" />
         </geometry>
-        <material name="red" />
+        <color rgba="1 1 0 1"/>
       </visual>
     </link>
     <joint name="camera_optical_joint" type="fixed">
-      <origin xyz="0 0 0" rpy="${-pi/2} 0 ${-pi/2}" />
+      <origin xyz="0 0 0" rpy="${-pi/2} 0 ${-90 * pi / 180}" />
       <parent link="camera_link" />
       <child link="camera_link_optical" />

File: ar_description/urdf/ar_gazebo.urdf.xacro (robot description, xacro)
@@ -19,4 +19,6 @@
     calibrate="False"
     joint_offset_parameters_file="$(find ar_hardware_interface)/config/joint_offsets.yaml"
+    joint_velocity_parameters_file="$(find ar_hardware_interface)/config/joint_velocities.yaml"
+    joint_acceleration_parameters_file="$(find ar_hardware_interface)/config/joint_accelerations.yaml"
   />
   <xacro:ar_gripper_ros2_control

File: ar_hardware_interface/urdf/ar.urdf.xacro (robot description, xacro)
@@ -17,4 +17,6 @@
     calibrate="$(arg calibrate)"
     joint_offset_parameters_file="$(find ar_hardware_interface)/config/joint_offsets.yaml"
+    joint_velocity_parameters_file="$(find ar_hardware_interface)/config/joint_velocities.yaml"
+    joint_acceleration_parameters_file="$(find ar_hardware_interface)/config/joint_accelerations.yaml"
   />
   <xacro:if value="$(arg include_gripper)">
@@ -28,3 +30,6 @@
     />
   </xacro:if>
+  <xacro:include
+    filename="$(find ar_description)/urdf/ar_camera_macro.xacro" />
+  <xacro:ar_camera />
 </robot>

File: ar_moveit_config/srdf/ar_macro.srdf.xacro (robot description, xacro)
@@ -31,4 +31,12 @@
       <joint name="joint_6" value="0" />
     </group_state>
+    <group_state name="facing_left" group="ar_manipulator">
+      <joint name="joint_1" value="-0.9" />
+      <joint name="joint_2" value="0" />
+      <joint name="joint_3" value="0" />
+      <joint name="joint_4" value="0" />
+      <joint name="joint_5" value="0" />
+      <joint name="joint_6" value="0" />
+    </group_state>
     <disable_collisions link1="base_link" link2="link_1" reason="Adjacent" />
     <disable_collisions link1="link_1" link2="link_2" reason="Adjacent" />

File: ar_moveit_config/urdf/fake_ar.urdf.xacro (robot description, xacro)
@@ -16,4 +16,6 @@
     calibrate="False"
     joint_offset_parameters_file="$(find ar_hardware_interface)/config/joint_offsets.yaml"
+    joint_velocity_parameters_file="$(find ar_hardware_interface)/config/joint_velocities.yaml"
+    joint_acceleration_parameters_file="$(find ar_hardware_interface)/config/joint_accelerations.yaml"
   />
   <xacro:ar_gripper_ros2_control
